File: Platinen/Steuerplatine/WortuhrNeu.kicad_pcb (KiCad board)
At the start: 2 copper layers, 339 x 29 mm, 73 parts, among them J1 Conn_01x01_Pin, J2 PROG MODE, J3 UART FLOATING, J4 UART, SW1 PTS645Vx83-2LFS, SW2 PTS645Vx83-2LFS, U1 DIP6 Sockel für H11L1, U2 MCP1826-ADJE/ET, U3 Bluepill, U4 DS18B20, U5 DS3231 Module, U6 Arduino_Nano_Every, U7 ESP-07, X1 Conn_01x03_Pin, X10 Conn_01x03_Pin, X11 Conn_01x03_Pin, X12 Conn_01x03_Pin, X13 Conn_01x03_Pin, X14 Conn_01x03_Pin, X15 Conn_01x03_Pin, X16 Conn_01x03_Pin, X17 Conn_01x03_Pin, X18 Conn_01x03_Pin, X19 Conn_01x03_Pin, X2 Conn_01x03_Pin, X3 Conn_01x03_Pin, X4 Conn_01x03_Pin, X5 Conn_01x03_Pin, X6 Conn_01x03_Pin, X7 Conn_01x03_Pin, X8 Conn_01x03_Pin, X9 Conn_01x03_Pin

Commit message: added trotec template
Changed lines of the file:
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@@
 		(tags "Resistor Axial_DIN0207 series Axial Horizontal pin pitch 10.16mm 0.25W = 1/4W length 6.3mm diameter 2.5mm")
 		(property "Reference" "R15"
-			(at 12.83 -3 90)
+			(at 12.78 -0.25 90)
 			(layer "F.SilkS")
 			(effects
@@
 		(tags "Resistor Axial_DIN0207 series Axial Horizontal pin pitch 10.16mm 0.25W = 1/4W length 6.3mm diameter 2.5mm")
 		(property "Reference" "R13"
-			(at -2.75 -3 90)
+			(at -2.71744 0.153932 90)
 			(layer "F.SilkS")
 			(effects
@@
 		)
 	)
+	(dimension
+		(type orthogonal)
+		(layer "Edge.Cuts")
+		(pts
+			(xy 41.75 169.489377) (xy 41.75 140.5)
+		)
+		(height -1.45)
+		(orientation 1)
+		(format
+			(prefix "")
+			(suffix "")
+			(units 3)
+			(units_format 1)
+			(precision 4)
+		)
+		(style
+			(thickness 0.05)
+			(arrow_length 1.27)
+			(text_position_mode 0)
+			(arrow_direction outward)
+			(extension_height 0.58642)
+			(extension_offset 0.5)
+			(keep_text_aligned yes)
+		)
+		(gr_text "28.9894 mm"
+			(at 39.15 154.994688 90)
+			(layer "Edge.Cuts")
+			(effects
+				(font
+					(size 1 1)
+					(thickness 0.15)
+				)
+			)
+		)
+	)
