File: Platinen/Kombiplatine SMD/WortuhrNeu.kicad_pcb (KiCad board)
At the start: 2 copper layers, 339 x 40.5 mm, 98 parts, among them J1 Conn_01x01_Pin, J2 PROG MODE, J3 UART FLOATING, J4 UART, J5 Eingangsbuchse, SW1 PTS645Vx83-2LFS, SW2 PTS645Vx83-2LFS, U2 MCP1826-ADJE/ET, U3 Bluepill, U4 DS18B20, U6 Arduino_Nano_Every, U7 ESP-07, U8 Generic DCDC, U9 TP582, X1 Conn_01x03_Pin, X10 Conn_01x03_Pin, X11 Conn_01x03_Pin, X12 Conn_01x03_Pin, X13 Conn_01x03_Pin, X14 Conn_01x03_Pin, X15 Conn_01x03_Pin, X16 Conn_01x03_Pin, X17 Conn_01x03_Pin, X18 Conn_01x03_Pin, X19 Conn_01x03_Pin, X2 Conn_01x03_Pin, X20 Conn_01x03_Pin, X21 Conn_01x03_Pin, X22 Conn_01x03_Pin, X23 Conn_01x03_Pin, X24 Conn_01x03_Pin, X25 Conn_01x03_Pin, X26 Conn_01x03_Pin, X27 Conn_01x03_Pin, X28 Conn_01x03_Pin, X29 Conn_01x03_Pin, X3 Conn_01x03_Pin, X30 Conn_01x03_Pin, X31 Conn_01x03_Pin, X32 Conn_01x03_Pin, X33 Conn_01x03_Pin, X34 Conn_01x03_Pin, X35 Conn_01x03_Pin, X36 Conn_01x03_Pin, X37 Conn_01x03_Pin, X38 Conn_01x03_Pin, X4 Conn_01x03_Pin, X5 Conn_01x03_Pin, X6 Conn_01x03_Pin, X7 Conn_01x03_Pin, X8 Conn_01x03_Pin, X9 Conn_01x03_Pin

Commit message: Implemented changes made for 2026 version, added second dcdc
Other:
- outline, holes or cut-outs redrawn
