File: Platinen/Kombiplatine THT/WortuhrNeu.kicad_pcb (KiCad board)
At the start: 2 copper layers, 339 x 58 mm, 101 parts, among them J1 Conn_01x01_Pin, J2 PROG MODE, J3 UART FLOATING, J4 UART, J5 Eingangsbuchse, SW1 PTS645Vx83-2LFS, SW2 PTS645Vx83-2LFS, U2 MCP1826-ADJE/ET, U3 Bluepill, U4 DS18B20, U6 Arduino_Nano_Every, U7 ESP-07, U8 Generic DCDC, U9 TP582, X1 Conn_01x03_Pin, X10 Conn_01x03_Pin, X11 Conn_01x03_Pin, X12 Conn_01x03_Pin, X13 Conn_01x03_Pin, X14 Conn_01x03_Pin, X15 Conn_01x03_Pin, X16 Conn_01x03_Pin, X17 Conn_01x03_Pin, X18 Conn_01x03_Pin, X19 Conn_01x03_Pin, X2 Conn_01x03_Pin, X20 Conn_01x03_Pin, X21 Conn_01x03_Pin, X22 Conn_01x03_Pin, X23 Conn_01x03_Pin, X24 Conn_01x03_Pin, X25 Conn_01x03_Pin, X26 Conn_01x03_Pin, X27 Conn_01x03_Pin, X28 Conn_01x03_Pin, X29 Conn_01x03_Pin, X3 Conn_01x03_Pin, X30 Conn_01x03_Pin, X31 Conn_01x03_Pin, X32 Conn_01x03_Pin, X33 Conn_01x03_Pin, X34 Conn_01x03_Pin, X35 Conn_01x03_Pin, X36 Conn_01x03_Pin, X37 Conn_01x03_Pin, X38 Conn_01x03_Pin, X4 Conn_01x03_Pin, X5 Conn_01x03_Pin, X6 Conn_01x03_Pin, X7 Conn_01x03_Pin, X8 Conn_01x03_Pin, X9 Conn_01x03_Pin

Commit message: Implemented changes made for 2026 version, added second dcdc
Parts:
- added U10: Generic DCDC, Converter_DCDC:Converter_DCDC_RECOM_R-78B-2.0_THT, F.Cu at (208.3, 182.5)
- moved U8 8.39 mm to (336.2, 183.2), turned to 0 degrees
Connections:
- C15 pad 1: +5V -> +5V4
- C17 pad 1: +5V -> +5V4
- U6 pad 27: +5V -> +5V4
- U6 pad 30: +5V -> +5V4
- X11 pad 3: +5V -> +5V4
- X12 pad 3: +5V -> +5V4
- X13 pad 1: +5V -> +5V4
- X14 pad 3: +5V -> +5V4
- X15 pad 1: +5V -> +5V4
- X16 pad 1: +5V -> +5V4
- X17 pad 1: +5V -> +5V4
- X18 pad 3: +5V -> +5V4
- X19 pad 3: +5V -> +5V4
- X29 pad 3: +5V2 -> +5V3
- X30 pad 1: +5V2 -> +5V3
- X31 pad 3: +5V2 -> +5V3
- X32 pad 1: +5V2 -> +5V3
- X33 pad 3: +5V2 -> +5V3
- X34 pad 1: +5V2 -> +5V3
- X35 pad 3: +5V2 -> +5V3
- X36 pad 1: +5V2 -> +5V3
- X37 pad 3: +5V2 -> +5V3
- X38 pad 1: +5V2 -> +5V3
- X9 pad 1: +5V -> +5V4
Routing:
- net +5V: track 372.3 -> 164.8 mm
- net +5V4: track 0.00 -> 190.3 mm, vias 0 -> 1
- net Net-(U10-IN): track 22.2 -> 173.4 mm
- net GND: track 76.0 -> 80.6 mm
- added copper zone on B.Cu, net +5V3
Other:
- board text removed: "HTTPS://GITHU"
- board text removed: "HTTPS://GITHUB.COM"
- board text removed: "HTTPS://GITHUB.COM/RT-CUSTO"
- board text removed: "HTTPS://GITHUB.COM/RT-CUSTOMZ/WORTUHR"
- board text removed: "HTTPS://GITHUB.COM/RT-CUSTOMZ/WORTUHR-MINI"
- board text removed: "HTTPS://GITHUB.COM/RT-CUSTOMZ/WORTUHR-MINI HTT"
