File: Platinen/Kombiplatine THT/WortuhrNeu.kicad_pcb (KiCad board)
At the start: 2 copper layers, 339 x 58 mm, 102 parts, among them J1 Conn_01x01_Pin, J2 PROG MODE, J3 UART FLOATING, J4 UART, J5 Eingangsbuchse, SW1 PTS645Vx83-2LFS, SW2 PTS645Vx83-2LFS, U10 Generic DCDC, U2 MCP1826-ADJE/ET, U3 Bluepill, U4 DS18B20, U6 Arduino_Nano_Every, U7 ESP-07, U8 Generic DCDC, U9 TP582, X1 Conn_01x03_Pin, X10 Conn_01x03_Pin, X11 Conn_01x03_Pin, X12 Conn_01x03_Pin, X13 Conn_01x03_Pin, X14 Conn_01x03_Pin, X15 Conn_01x03_Pin, X16 Conn_01x03_Pin, X17 Conn_01x03_Pin, X18 Conn_01x03_Pin, X19 Conn_01x03_Pin, X2 Conn_01x03_Pin, X20 Conn_01x03_Pin, X21 Conn_01x03_Pin, X22 Conn_01x03_Pin, X23 Conn_01x03_Pin, X24 Conn_01x03_Pin, X25 Conn_01x03_Pin, X26 Conn_01x03_Pin, X27 Conn_01x03_Pin, X28 Conn_01x03_Pin, X29 Conn_01x03_Pin, X3 Conn_01x03_Pin, X30 Conn_01x03_Pin, X31 Conn_01x03_Pin, X32 Conn_01x03_Pin, X33 Conn_01x03_Pin, X34 Conn_01x03_Pin, X35 Conn_01x03_Pin, X36 Conn_01x03_Pin, X37 Conn_01x03_Pin, X38 Conn_01x03_Pin, X4 Conn_01x03_Pin, X5 Conn_01x03_Pin, X6 Conn_01x03_Pin, X7 Conn_01x03_Pin, X8 Conn_01x03_Pin, X9 Conn_01x03_Pin

Commit message: Edited descriptors in Kicad and updated iBom
Parts:
- C1: value 47u -> 47u 25V
- C13: value 47u -> 47uF 25V
- C20, C3, C4, C7, C9: value 10u -> 1u
- U5: value ~ -> DS3231 Module
- U6: value Arduino_Nano_Every -> Arduino nano
- U7: value ESP-07 -> ESP8266 Module
Other:
- board text added: "1u"
- board text added: "STM32-BLUEPILL"
- board text removed: "10u"
- board text removed: "STM32-BLACKPILL"
Changed lines of the file:
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@@
 			)
 		)
-		(property "Description" "Resistor"
+		(property "Description" "Resistor Axial 250mW"
 			(at 0 0 0)
 			(layer "F.Fab")
@@
 			)
 		)
-		(property "Description" "Resistor"
+		(property "Description" "Resistor Axial 250mW"
 			(at 0 0 0)
 			(unlocked yes)
@@
 			)
 		)
-		(property "Value" "10u"
+		(property "Value" "1u"
 			(at 2.5 2.5 90)
 			(layer "F.Fab")
@@
 			)
 		)
-		(property "Description" "Unpolarized capacitor, small symbol"
+		(property "Description" "Kerko THT"
 			(at 0 0 270)
 			(unlocked yes)
@@
 			)
 		)
-		(property "Value" "10u"
+		(property "Value" "1u"
 			(at 2.5 2.5 90)
 			(layer "F.Fab")
@@
 			)
 		)
-		(property "Description" "Unpolarized capacitor, small symbol"
+		(property "Description" "Kerko THT"
 			(at 0 0 90)
 			(unlocked yes)
@@
 			)
 		)
-		(property "Value" "10u"
+		(property "Value" "1u"
 			(at 2.5 2.5 90)
 			(layer "F.Fab")
@@
 			)
 		)
-		(property "Description" "Unpolarized capacitor, small symbol"
+		(property "Description" "Kerko THT"
 			(at 0 0 90)
 			(unlocked yes)
@@
 			)
 		)
-		(property "Description" "Unpolarized capacitor, small symbol"
+		(property "Description" "Kerko THT"
 			(at 0 0 90)
 			(layer "F.Fab")
@@
 			)
 		)
-		(property "Value" "Arduino_Nano_Every"
+		(property "Value" "Arduino nano"
 			(at 8.89 19.05 0)
 			(layer "F.Fab")
@@
 			)
 		)
-		(property "Description" "Arduino Nano Every"
+		(property "Description" "Optional Arduino Nano for hijacking the WS2812 Signal and broadcasting your own"
 			(at 0 0 90)
 			(unlocked yes)
@@
 			)
 		)
-		(property "Value" "~"
+		(property "Value" "DS3231 Module"
 			(at 0.2 7.6 0)
 			(unlocked yes)
@@
 			)
 		)
-		(property "Description" ""
+		(property "Description" "DS3231 Module with integrated AT24CS32, 2032 lithium cell"
 			(at -16.2 6.75 0)
 			(unlocked yes)
@@
 			)
 		)
-		(property "Description" "Resistor"
+		(property "Description" "Resistor Axial 250mW"
 			(at 0 0 0)
 			(layer "F.Fab")
@@
 			)
 		)
-		(attr through_hole)
+		(attr through_hole exclude_from_bom dnp)
 		(duplicate_pad_numbers_are_jumpers no)
 		(fp_line
@@
 			)
 		)
-		(property "Description" "Resistor"
+		(property "Description" "Resistor Axial 250mW"
 			(at 0 0 90)
 			(unlocked yes)
@@
 			)
 		)
-		(attr through_hole)
+		(attr through_hole exclude_from_bom dnp)
 		(duplicate_pad_numbers_are_jumpers no)
 		(fp_line
@@
 			)
 		)
-		(property "Description" "Resistor"
+		(property "Description" "Resistor Axial 250mW"
 			(at 0 0 90)
 			(layer "F.Fab")
@@
 			)
 		)
-		(property "Description" "Resistor"
+		(property "Description" "Resistor Axial 250mW"
 			(at 0 0 270)
 			(unlocked yes)
@@
 			)
 		)
-		(property "Description" "Unpolarized capacitor, small symbol"
+		(property "Description" "Kerko THT"
 			(at 0 0 270)
 			(unlocked yes)
@@
 			)
 		)
-		(attr smd)
+		(attr smd exclude_from_bom dnp)
 		(duplicate_pad_numbers_are_jumpers no)
 		(fp_line
@@
 			)
 		)
-		(property "Description" "Resistor"
+		(property "Description" "Resistor Axial 250mW"
 			(at 0 0 270)
 			(unlocked yes)
@@
 		(tags "CP Radial series Radial pin pitch 5.00mm  diameter 10mm Electrolytic Capacitor")
 		(property "Reference" "C13"
-			(at 2.367677 6.25 270)
+			(at 2.367677 6.25 90)
 			(layer "F.SilkS")
 			(effects
@@
 			)
 		)
-		(property "Value" "47u"
+		(property "Value" "47uF 25V"
 			(at 2.5 6.25 90)
 			(layer "F.Fab")
@@
 			)
 		)
-		(property "Description" "Polarized capacitor"
+		(property "Description" "Polarized electrolytic capacitor 5mm pitch"
 			(at 0 0 270)
 			(unlocked yes)
@@
 			)
 		)
-		(property "Description" "Resistor"
+		(property "Description" "Resistor Axial 250mW"
 			(at 0 0 270)
 			(unlocked yes)
@@
 			)
 		)
-		(property "Description" "Unpolarized capacitor, small symbol"
+		(property "Description" "Kerko THT"
 			(at 0 0 90)
 			(unlocked yes)
@@
 			)
 		)
-		(property "Description" "2A Step-Down DC/DC-Regulator, 6.5-32V input, 5.0V fixed Output Voltage, LM78xx replacement, -40°C to +85°C, SIP3"
+		(property "Description" "2A Step-Down DC/DC-Regulator, 6.5-32V input, 5.0V fixed Output Voltage -40°C to +85°C, SIP3"
 			(at 0 0 0)
 			(unlocked yes)
@@
 			)
 		)
-		(property "Description" "Unpolarized capacitor, small symbol"
+		(property "Description" "Kerko THT"
 			(at 0 0 270)
 			(unlocked yes)
@@
 			)
 		)
-		(property "Description" "Unpolarized capacitor, small symbol"
+		(property "Description" "Kerko THT"
 			(at 0 0 90)
 			(layer "F.Fab")
@@
 			)
 		)
-		(property "Value" "ESP-07"
+		(property "Value" "ESP8266 Module"
 			(at 0 9.6 90)
 			(layer "F.Fab")
@@
 			)
 		)
-		(property "Description" "802.11 b/g/n Wi-Fi Module"
+		(property "Description" "ESP-12F"
 			(at 0 0 270)
 			(unlocked yes)
@@
 			)
 		)
-		(property "Description" "Unpolarized capacitor, small symbol"
+		(property "Description" "Kerko THT"
 			(at 0 0 90)
 			(unlocked yes)
@@
 			)
 		)
-		(property "Value" "10u"
+		(property "Value" "1u"
 			(at 2.5 2.5 90)
 			(layer "F.Fab")
@@
 			)
 		)
-		(property "Description" "Unpolarized capacitor, small symbol"
+		(property "Description" "Kerko THT"
 			(at 0 0 90)
 			(unlocked yes)
@@
 			)
 		)
-		(property "Description" "Unpolarized capacitor, small symbol"
+		(property "Description" "Kerko THT"
 			(at 0 0 90)
 			(unlocked yes)
@@
 			)
 		)
-		(property "Value" "10u"
+		(property "Value" "1u"
 			(at 2.5 2.5 90)
 			(layer "F.Fab")
@@
 			)
 		)
-		(property "Description" "Unpolarized capacitor, small symbol"
+		(property "Description" "Kerko THT"
 			(at 0 0 270)
 			(unlocked yes)
@@
 			)
 		)
-		(property "Description" "Unpolarized capacitor, small symbol"
+		(property "Description" "Kerko THT"
 			(at 0 0 90)
 			(unlocked yes)
@@
 			)
 		)
-		(property "Description" "Resistor"
+		(property "Description" "Resistor Axial 250mW"
 			(at 0 0 180)
 			(unlocked yes)
@@
 			)
 		)
-		(property "Description" "Unpolarized capacitor, small symbol"
+		(property "Description" "Kerko THT"
 			(at 0 0 270)
 			(unlocked yes)
@@
 			)
 		)
-		(property "Description" "2A Step-Down DC/DC-Regulator, 6.5-32V input, 5.0V fixed Output Voltage, LM78xx replacement, -40°C to +85°C, SIP3"
+		(property "Description" "2A Step-Down DC/DC-Regulator, 6.5-32V input, 5.0V fixed Output Voltage -40°C to +85°C, SIP3"
 			(at 0 0 0)
 			(unlocked yes)
@@
 			)
 		)
-		(property "Description" "Unpolarized capacitor, small symbol"
+		(property "Description" "Kerko THT"
 			(at 0 0 90)
 			(layer "F.Fab")
@@
 			)
 		)
-		(property "Description" "Resistor"
+		(property "Description" "Resistor Axial 250mW"
 			(at 0 0 270)
 			(unlocked yes)
@@
 			)
 		)
-		(property "Description" "Unpolarized capacitor, small symbol"
+		(property "Description" "Kerko THT"
 			(at 0 0 90)
 			(layer "F.Fab")
@@
 			)
 		)
-		(property "Description" "Resistor"
+		(property "Description" "Resistor Axial 250mW"
 			(at 0 0 90)
 			(unlocked yes)
@@
 			)
 		)
-		(property "Description" "Resistor"
+		(property "Description" "Resistor Axial 250mW"
 			(at 0 0 90)
 			(layer "F.Fab")
@@
 			)
 		)
-		(property "Value" "47u"
+		(property "Value" "47u 25V"
 			(at 2.5 6.25 90)
 			(layer "F.Fab")
@@
 			)
 		)
-		(property "Description" "Polarized capacitor"
+		(property "Description" "Polarized electrolytic capacitor 5mm pitch"
 			(at 0 0 90)
 			(unlocked yes)
@@
 			)
 		)
-		(property "Description" "Resistor"
+		(property "Description" "Resistor Axial 250mW"
 			(at 0 0 90)
 			(unlocked yes)
@@
 			)
 		)
-		(property "Description" "Unpolarized capacitor, small symbol"
+		(property "Description" "Kerko THT"
 			(at 0 0 0)
 			(layer "F.Fab")
@@
 			)
 		)
-		(property "Description" "Resistor"
+		(property "Description" "Resistor Axial 250mW"
 			(at 0 0 90)
 			(layer "F.Fab")
@@
 			)
 		)
-		(property "Description" "Unpolarized capacitor, small symbol"
+		(property "Description" "Kerko THT"
 			(at 0 0 90)
 			(unlocked yes)
@@
 			)
 		)
-		(property "Description" ""
+		(property "Description" "STM32F103C8T6 Bluepill"
 			(at 0.25 1.75 90)
 			(unlocked yes)
@@
 			)
 		)
-		(property "Description" "Resistor"
+		(property "Description" "Resistor Axial 250mW"
 			(at 0 0 270)
 			(unlocked yes)
@@
 	)
 	(gr_rect
-		(start 114.75 153)
-		(end 120.5 159.5)
+		(start 162.675 153.55)
+		(end 168.425 160.05)
 		(stroke
 			(width 0.2)
@@
 	)
 	(gr_line
-		(start 115.5 150.5)
-		(end 115.5 153)
-		(stroke
-			(width 0.15)
-			(type default)
-		)
-		(layer "F.SilkS")
-	)
-	(gr_line
-		(start 115.5 159.5)
-		(end 115.5 162.25)
+		(start 166.45 151.05)
+		(end 166.45 153.55)
 		(stroke
 			(width 0.15)
@@
 	)
 	(gr_line
-		(start 166.434 150.83)
-		(end 166.434 163.17)
+		(start 166.45 160.1)
+		(end 166.45 162.85)
 		(stroke
 			(width 0.15)
@@
 		)
 	)
-	(gr_text "STM32-BLACKPILL"
+	(gr_text "STM32-BLUEPILL"
 		(at 135.25 162.5 0)
 		(layer "F.SilkS" knockout)
@@
 	)
 	(gr_text "USB"
-		(at 116.5 158 90)
+		(at 164.425 158.55 90)
 		(layer "F.SilkS")
 		(effects
@@
 		)
 	)
-	(gr_text "10u"
+	(gr_text "1u"
 		(at 77.409522 156.012314 90)
 		(layer "F.SilkS" knockout)
@@
 		)
 	)
-	(gr_text "10u"
+	(gr_text "1u"
 		(at 80.338929 155.968808 90)
 		(layer "F.SilkS" knockout)
@@
 		)
 	)
-	(gr_text "10u"
+	(gr_text "1u"
 		(at 109.830822 164.778684 90)
 		(layer "F.SilkS" knockout)
@@
 		)
 	)
-	(gr_text "10u"
+	(gr_text "1u"
 		(at 109.930725 156.486751 90)
 		(layer "F.SilkS" knockout)
@@
 		)
 	)
-	(gr_text "10u"
+	(gr_text "1u"
 		(at 354.845028 154.257935 90)
 		(layer "F.SilkS" knockout)
@@
 	)
 	(group ""
-		(members "3531bed8-6fbc-4c74-816d-5dcff8cafc15" "b4ce3a27-e8cb-4c53-b3e4-2adce5909061")
-	)
-	(group ""
-		(members "081a1cbc-33a2-4753-a9d1-02354fd66025" "dd664a53-b100-49bf-aee6-42a074142da5")
+		(members "081a1cbc-33a2-4753-a9d1-02354fd66025")
 	)
 	(embedded_fonts no)
