File: Platinen/Kombiplatine THT/WortuhrNeu.kicad_sch (KiCad schematic)
At the start: 101 parts, among them J1 Conn_01x01_Pin, J2 PROG MODE, J3 UART FLOATING, J4 UART, J5 Eingangsbuchse, SW1 PTS645Vx83-2LFS, SW2 PTS645Vx83-2LFS, U2 MCP1826-ADJE/ET, U3 Bluepill, U4 DS18B20, U6 Arduino_Nano_Every, U7 ESP-07, U8 Generic DCDC, U9 TP582, X1 Conn_01x03_Pin, X10 Conn_01x03_Pin, X11 Conn_01x03_Pin, X12 Conn_01x03_Pin, X13 Conn_01x03_Pin, X14 Conn_01x03_Pin, X15 Conn_01x03_Pin, X16 Conn_01x03_Pin, X17 Conn_01x03_Pin, X18 Conn_01x03_Pin, X19 Conn_01x03_Pin, X2 Conn_01x03_Pin, X20 Conn_01x03_Pin, X21 Conn_01x03_Pin, X22 Conn_01x03_Pin, X23 Conn_01x03_Pin, X24 Conn_01x03_Pin, X25 Conn_01x03_Pin, X26 Conn_01x03_Pin, X27 Conn_01x03_Pin, X28 Conn_01x03_Pin, X29 Conn_01x03_Pin, X3 Conn_01x03_Pin, X30 Conn_01x03_Pin, X31 Conn_01x03_Pin, X32 Conn_01x03_Pin, X33 Conn_01x03_Pin, X34 Conn_01x03_Pin, X35 Conn_01x03_Pin, X36 Conn_01x03_Pin, X37 Conn_01x03_Pin, X38 Conn_01x03_Pin, X4 Conn_01x03_Pin, X5 Conn_01x03_Pin, X6 Conn_01x03_Pin, X7 Conn_01x03_Pin, X8 Conn_01x03_Pin, X9 Conn_01x03_Pin

Commit message: Implemented changes made for 2026 version, added second dcdc
Parts:
- added U10: Generic DCDC, Converter_DCDC:Converter_DCDC_RECOM_R-78B-2.0_THT, symbol Regulator_Switching:R-78B5.0-2.0
Connections:
- net +5V: no longer C15.1, C17.1, J4.1 (Pin_1), U6.27 (+5V), U6.30 (VIN), X11.3 (Pin_3), X12.3 (Pin_3), X13.1 (Pin_1), X14.3 (Pin_3), X15.1 (Pin_1), X16.1 (Pin_1), X17.1 (Pin_1), X18.3 (Pin_3), X19.3 (Pin_3), X9.1 (Pin_1)
- net +5V2: no longer X29.3 (Pin_3), X30.1 (Pin_1), X31.3 (Pin_3), X32.1 (Pin_1), X33.3 (Pin_3), X34.1 (Pin_1), X35.3 (Pin_3), X36.1 (Pin_1), X37.3 (Pin_3), X38.1 (Pin_1)
- net GND2: now also U10.2 (GND)
- net at TH1.2, U8.1 (IN): now also U10.1 (IN)
- new net +5V3: U10.3 (OUT), X29.3 (Pin_3), X30.1 (Pin_1), X31.3 (Pin_3), X32.1 (Pin_1), X33.3 (Pin_3), X34.1 (Pin_1), X35.3 (Pin_3), X36.1 (Pin_1), X37.3 (Pin_3), X38.1 (Pin_1)
- new net +5V4: C15.1, C17.1, J4.1 (Pin_1), U6.27 (+5V), U6.30 (VIN), X11.3 (Pin_3), X12.3 (Pin_3), X13.1 (Pin_1), X14.3 (Pin_3), X15.1 (Pin_1), X16.1 (Pin_1), X17.1 (Pin_1), X18.3 (Pin_3), X19.3 (Pin_3), X9.1 (Pin_1)

Commit message: Edited descriptors in Kicad and updated iBom
Parts:
- added J6, J7: Conn_01x08_Pin, Connector_PinHeader_2.00mm:PinHeader_1x08_P2.00mm_Vertical, symbol Connector:Conn_01x08_Pin
- added J8, J9: Conn_01x08_Socket, Connector_PinSocket_2.00mm:PinSocket_1x08_P2.00mm_Vertical, symbol Connector:Conn_01x08_Socket
- C1: value 47u -> 47u 25V
- C13: value 47u -> 47uF 25V
- C19, R1, R6: now not fitted; now left out of the parts list
- C20, C3, C4, C7, C9: value 10u -> 1u
- J1: KiLib_Generator (none) -> connector/pin_header_socket
- U5: value (none) -> DS3231 Module
- U6: value Arduino_Nano_Every -> Arduino nano
- U7: value ESP-07 -> ESP8266 Module
Connections:
- net +5V: now also J4.1 (Pin_1)
- net +5V4: no longer J4.1 (Pin_1)
- no-connect marks 58 -> 90
